File: 32u4 plus 16LEDs/FabDisPendant.brd (EAGLE design)
At the start: 76.2 x 54.2 mm, 70 parts, among them IC1 MPR121, J2 AVR_SPI_PRG_6PTH, U3 ATMEGA32U4, Y1 16MHz

Commit message: Checkin prior to autorouting
Parts:
- removed D3: Green, SparkFun:LED-0603
- removed R6: 330, SparkFun:0603-RES
- moved X2 65.9 mm to (50.2, 2.79), turned to 90 degrees
- moved D2 63.6 mm to (43.4, 9.78)
- moved F1 58.5 mm to (47.4, 8.13), turned to 180 degrees
- moved R11 58.1 mm to (46.6, 13.3), turned to 270 degrees
- moved R5 58.0 mm to (52.7, 8.51), turned to 270 degrees
- moved R7 57.8 mm to (50.4, 8.51), turned to 270 degrees
- moved LED1 56.8 mm to (48.4, 13.5), turned to 180 degrees
- moved C25 55.4 mm to (47.6, 10.3), turned to 0 degrees
- moved 7803-??? 20.9 mm to (56.1, 30.7)
- moved C32 20.3 mm to (47.8, 33.3)
- moved C31 19.9 mm to (47.8, 27.4)
- moved C29 16.6 mm to (41.1, 13.0), turned to 180 degrees
- moved U$1 16.1 mm to (33.8, 38.8)
- moved 7805 14.6 mm to (33.3, 14.7), turned to 90 degrees
- moved C26 10.1 mm to (38.6, 28.3), turned to 270 degrees
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Connections:
- removed net N$24: D3.C, R6.2
- removed net TXLED: R6.1, U3.22
- net 5V: no longer D3.A
Routing:
- net 5V: track 243.0 -> 333.1 mm
- net RAW: track 0.00 -> 41.1 mm
- net 3.3V: track 1.99 -> 36.2 mm
- net RESET: track 0.00 -> 24.0 mm
- net GND: track 0.00 -> 17.9 mm
- net USBVCC: track 8.26 -> 4.17 mm
- net N$25: track 0.00 -> 2.87 mm
- net N$19: track 0.00 -> 2.79 mm
- net AREF: track 0.00 -> 2.32 mm
- net N$18: track 5.25 -> 7.28 mm
- net N$17: track 8.41 -> 10.4 mm
- net N$1: track 0.00 -> 1.88 mm
- net N$38: track 0.00 -> 1.78 mm

Commit message: More improvements, checkin before rearrangement
Parts:
- moved C28 1.52 mm to (53.8, 22.4)
Routing:
- net USBVCC: track 4.17 -> 5.00 mm
- net 5V: track 333.1 -> 332.3 mm
Changed lines of the file:
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@@
 <element name="C27" library="SparkFun" package="0603-CAP" value="0.1uF" x="51.435" y="15.367" rot="R180"/>
 <element name="R1" library="SparkFun" package="0603-RES" value="75k" x="53.975" y="12.7254" rot="R90"/>
-<element name="C28" library="SparkFun" package="0603-CAP" value="0.1uF" x="53.848" y="20.9042" rot="R90"/>
+<element name="C28" library="SparkFun" package="0603-CAP" value="0.1uF" x="53.848" y="22.4282" rot="R90"/>
 <element name="JP3" library="SparkFun" package="1X12" value="Electrodes" x="60.579" y="29.972" rot="R270"/>
 <element name="R3" library="SparkFun" package="0603-RES" value="4.7k" x="50.292" y="17.907" rot="R180"/>
@@
 <wire x1="53.9115" y1="6.9215" x2="53.9115" y2="11.8119" width="0.254" layer="1"/>
 <wire x1="53.9115" y1="11.8119" x2="53.975" y2="11.8754" width="0.254" layer="1"/>
-<wire x1="21.3325" y1="47.229" x2="21.097" y2="47.229" width="0.254" layer="1"/>
-<wire x1="21.097" y1="47.229" x2="19.812" y2="48.514" width="0.254" layer="1"/>
-<wire x1="19.812" y1="48.514" x2="19.089" y2="48.514" width="0.254" layer="1"/>
-<wire x1="19.089" y1="48.514" x2="18.542" y2="48.475" width="0.254" layer="1"/>
-<wire x1="23.174" y1="50.5655" x2="23.174" y2="51.668" width="0.254" layer="1"/>
-<wire x1="23.174" y1="51.668" x2="22.645" y2="52.705" width="0.254" layer="1"/>
 <wire x1="27.118" y1="50.0725" x2="27.118" y2="51.054" width="0.254" layer="1"/>
 <wire x1="27.118" y1="51.054" x2="28.702" y2="51.054" width="0.254" layer="1"/>
 <wire x1="28.702" y1="51.054" x2="28.702" y2="49.201" width="0.254" layer="1"/>
 <wire x1="28.702" y1="49.201" x2="28.4825" y2="49.201" width="0.254" layer="1"/>
+<wire x1="21.3325" y1="47.229" x2="19.788" y2="47.229" width="0.254" layer="1"/>
+<wire x1="19.788" y1="47.229" x2="18.542" y2="48.475" width="0.254" layer="1"/>
+<wire x1="23.174" y1="50.5655" x2="23.174" y2="52.176" width="0.254" layer="1"/>
+<wire x1="23.174" y1="52.176" x2="22.645" y2="52.705" width="0.254" layer="1"/>
 <wire x1="25.146" y1="46.736" x2="24.16" y2="43.3995" width="0" layer="19" extent="1-1"/>
 </signal>
@@
 <wire x1="32.258" y1="20.828" x2="32.258" y2="30.988" width="0.8128" layer="16"/>
 <wire x1="32.258" y1="17.272" x2="35.814" y2="17.272" width="0.8128" layer="1"/>
-<wire x1="23.667" y1="43.3995" x2="23.622" y2="43.4445" width="0.254" layer="1"/>
-<wire x1="23.622" y1="43.4445" x2="23.622" y2="44.704" width="0.254" layer="1"/>
-<wire x1="23.622" y1="44.704" x2="23.682" y2="44.764" width="0.254" layer="1"/>
-<wire x1="23.682" y1="44.764" x2="28.4825" y2="44.764" width="0.254" layer="1"/>
 <wire x1="22.681" y1="50.0725" x2="22.681" y2="49.276" width="0.254" layer="1"/>
 <wire x1="22.681" y1="49.276" x2="27.686" y2="49.276" width="0.254" layer="1"/>
@@
 <wire x1="9.1685" y1="35.306" x2="10.3115" y2="36.449" width="0.254" layer="1"/>
 <wire x1="10.3115" y1="36.449" x2="14.732" y2="36.449" width="0.254" layer="1"/>
+<wire x1="23.667" y1="43.3995" x2="23.667" y2="44.764" width="0.254" layer="1"/>
+<wire x1="23.667" y1="44.764" x2="27.686" y2="44.764" width="0.254" layer="1"/>
 <wire x1="28.702" y1="34.544" x2="23.667" y2="42.9065" width="0" layer="19" extent="1-16"/>
 </signal>
@@
 <contactref element="C20" pad="2"/>
 <contactref element="U3" pad="42"/>
-<wire x1="23.667" y1="50.5655" x2="23.667" y2="51.519" width="0.254" layer="1"/>
-<wire x1="23.667" y1="51.519" x2="24.345" y2="52.705" width="0.254" layer="1"/>
+<wire x1="23.667" y1="50.5655" x2="23.667" y2="52.027" width="0.254" layer="1"/>
+<wire x1="23.667" y1="52.027" x2="24.345" y2="52.705" width="0.254" layer="1"/>
 </signal>
 <signal name="RESET">
@@
 <contactref element="R11" pad="1"/>
 <contactref element="LED1" pad="A"/>
-<wire x1="46.609" y1="14.185" x2="47.344" y2="14.185" width="0.254" layer="1"/>
-<wire x1="47.344" y1="14.185" x2="48.387" y2="14.212" width="0.254" layer="1"/>
+<wire x1="46.609" y1="14.185" x2="46.636" y2="14.212" width="0.254" layer="1"/>
+<wire x1="46.636" y1="14.212" x2="48.387" y2="14.212" width="0.254" layer="1"/>
 </signal>
 <signal name="MISO">
@@
 <wire x1="36.322" y1="4.064" x2="35.814" y2="4.064" width="1.27" layer="16"/>
 <wire x1="35.814" y1="4.064" x2="35.814" y2="12.192" width="1.27" layer="16"/>
-<wire x1="39.878" y1="12.954" x2="35.814" y2="11.684" width="1.27" layer="16"/>
 <wire x1="35.814" y1="11.684" x2="35.814" y2="12.192" width="1.27" layer="16"/>
-<wire x1="39.878" y1="12.954" x2="49.022" y2="20.828" width="1.27" layer="16"/>
-<wire x1="49.022" y1="20.828" x2="49.022" y2="27.432" width="1.27" layer="16"/>
 <wire x1="53.594" y1="28.194" x2="52.832" y2="27.432" width="1.27" layer="16"/>
 <wire x1="52.832" y1="27.432" x2="49.022" y2="27.432" width="1.27" layer="16"/>
-<wire x1="42.284" y1="9.779" x2="39.878" y2="12.185" width="0.8128" layer="1"/>
-<wire x1="39.878" y1="12.185" x2="39.878" y2="12.954" width="0.8128" layer="1"/>
+<wire x1="35.814" y1="12.192" x2="39.116" y2="12.192" width="1.27" layer="16"/>
+<wire x1="39.116" y1="12.192" x2="39.878" y2="12.954" width="1.27" layer="16"/>
+<wire x1="39.878" y1="12.954" x2="49.022" y2="22.098" width="1.27" layer="16"/>
+<wire x1="49.022" y1="22.098" x2="49.022" y2="27.432" width="1.27" layer="16"/>
+<wire x1="42.284" y1="9.779" x2="39.878" y2="12.185" width="1.27" layer="1"/>
+<wire x1="39.878" y1="12.185" x2="39.878" y2="12.954" width="1.27" layer="1"/>
 </signal>
 <signal name="D9">
@@
 <contactref element="U3" pad="6"/>
 <contactref element="C24" pad="2"/>
-<wire x1="21.3325" y1="46.736" x2="19.089" y2="46.736" width="0.254" layer="1"/>
-<wire x1="19.089" y1="46.736" x2="18.542" y2="46.775" width="0.254" layer="1"/>
+<wire x1="21.3325" y1="46.736" x2="18.581" y2="46.736" width="0.254" layer="1"/>
+<wire x1="18.581" y1="46.736" x2="18.542" y2="46.775" width="0.254" layer="1"/>
 </signal>
 <signal name="USBVCC">
@@
 <contactref element="X2" pad="VBUS1"/>
 <contactref element="F1" pad="1"/>
-<wire x1="48.865" y1="6.2992" x2="48.865" y2="7.874" width="0.4064" layer="1"/>
-<wire x1="48.865" y1="7.874" x2="48.771" y2="8.128" width="0.4064" layer="1"/>
 <wire x1="48.517" y1="10.287" x2="48.475" y2="10.287" width="0.4064" layer="1"/>
 <wire x1="48.771" y1="8.128" x2="48.771" y2="9.991" width="0.4064" layer="1"/>
 <wire x1="48.771" y1="9.991" x2="48.475" y2="10.287" width="0.4064" layer="1"/>
+<wire x1="48.771" y1="8.128" x2="48.865" y2="8.034" width="0.4064" layer="1"/>
+<wire x1="48.865" y1="8.034" x2="48.865" y2="5.494" width="0.4064" layer="1"/>
 <wire x1="21.8095" y1="46.243" x2="21.8095" y2="48.708" width="0" layer="19" extent="1-1"/>
 <wire x1="48.475" y1="10.287" x2="21.8095" y2="46.243" width="0" layer="19" extent="1-1"/>
@@
 <vertex x="62.738" y="26.67"/>
 </polygon>
-<via x="63.754" y="15.24" extent="1-16" drill="0.508"/>
-<wire x1="60.579" y1="4.572" x2="63.754" y2="7.747" width="0.4064" layer="16"/>
-<wire x1="63.754" y1="7.747" x2="63.754" y2="15.24" width="0.4064" layer="16"/>
+<via x="64.008" y="15.24" extent="1-16" drill="0.508"/>
 <wire x1="55.52308125" y1="15.518940625" x2="55.52308125" y2="9.62791875" width="0.2032" layer="1"/>
 <wire x1="55.52308125" y1="9.62791875" x2="60.579" y2="4.572" width="0.2032" layer="1"/>
+<wire x1="60.579" y1="4.572" x2="64.008" y2="8.001" width="0.4064" layer="16"/>
+<wire x1="64.008" y1="8.001" x2="64.008" y2="15.24" width="0.4064" layer="16"/>
 </signal>
 <signal name="CAP0">
@@
 <contactref element="R4" pad="2"/>
 <contactref element="R3" pad="2"/>
-<wire x1="54.328159375" y1="18.2630625" x2="54.328159375" y2="19.574040625" width="0.2032" layer="1"/>
-<wire x1="54.328159375" y1="19.574040625" x2="53.848" y2="20.0542" width="0.2032" layer="1"/>
 <contactref element="U$5" pad="VDD"/>
 <contactref element="C32" pad="1"/>
@@
 <wire x1="52.07" y1="30.734" x2="50.8" y2="29.464" width="0.8128" layer="1"/>
 <wire x1="50.8" y1="29.464" x2="50.8" y2="24.638" width="0.8128" layer="1"/>
-<wire x1="50.8" y1="24.638" x2="49.442" y2="23.28" width="0.8128" layer="1"/>
+<wire x1="50.8" y1="24.638" x2="50.673" y2="24.511" width="0.8128" layer="1"/>
+<wire x1="50.673" y1="24.511" x2="49.442" y2="23.28" width="0.8128" layer="1"/>
 <wire x1="49.442" y1="23.28" x2="49.442" y2="22.479" width="0.8128" layer="1"/>
 <wire x1="49.442" y1="22.479" x2="49.442" y2="20.193" width="0.8128" layer="1"/>
 <wire x1="49.442" y1="20.193" x2="49.442" y2="17.907" width="0.8128" layer="1"/>
-<wire x1="53.848" y1="20.0542" x2="53.086" y2="20.8162" width="0.254" layer="1"/>
-<wire x1="53.086" y1="20.8162" x2="53.086" y2="23.114" width="0.254" layer="1"/>
-<wire x1="53.086" y1="23.114" x2="51.562" y2="24.638" width="0.254" layer="1"/>
-<wire x1="51.562" y1="24.638" x2="50.8" y2="24.638" width="0.254" layer="1"/>
 <wire x1="53.594" y1="30.734" x2="55.626" y2="30.734" width="0.8128" layer="16"/>
 <wire x1="55.626" y1="30.734" x2="56.204" y2="31.312" width="0.8128" layer="16"/>
@@
 <wire x1="52.07" y1="30.734" x2="49.53" y2="33.274" width="0.8128" layer="1"/>
 <wire x1="49.53" y1="33.274" x2="49.022" y2="33.274" width="0.8128" layer="1"/>
+<wire x1="50.927" y1="24.511" x2="50.673" y2="24.511" width="0.254" layer="1"/>
+<wire x1="53.848" y1="21.5782" x2="50.927" y2="24.4992" width="0.254" layer="1"/>
+<wire x1="50.927" y1="24.4992" x2="50.927" y2="24.511" width="0.254" layer="1"/>
+<wire x1="54.328159375" y1="18.2630625" x2="54.328159375" y2="21.098040625" width="0.2032" layer="1"/>
+<wire x1="54.328159375" y1="21.098040625" x2="53.848" y2="21.5782" width="0.2032" layer="1"/>
 </signal>
 <signal name="MPRIRQ">

Commit message: Substantial rearrangement
Parts:
- moved X2 58.7 mm to (2.29, 36.7), turned to 0 degrees
- moved PWR 56.7 mm to (3.56, 50.3), turned to 270 degrees
- moved R5 51.5 mm to (8.00, 34.2), turned to 180 degrees
- moved R7 50.8 mm to (8.00, 36.4), turned to 180 degrees
- moved F1 50.6 mm to (7.62, 39.5), turned to 90 degrees
- moved D2 47.8 mm to (9.27, 43.2), turned to 270 degrees
- moved C25 47.7 mm to (9.78, 39.2), turned to 270 degrees
- moved S1 46.3 mm to (49.5, 40.6)
- moved C29 43.4 mm to (12.4, 45.5), turned to 90 degrees
- moved LED1 43.1 mm to (13.0, 38.0), turned to 90 degrees
- moved 7805 43.1 mm to (14.2, 53.3), turned to 0 degrees
- moved R11 42.9 mm to (12.8, 39.8), turned to 180 degrees
- moved R2 41.3 mm to (49.6, 35.8), turned to 180 degrees
- moved U$1 38.2 mm to (45.5, 2.48)
- moved C30 35.5 mm to (18.0, 45.5), turned to 90 degrees
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Routing:
- net 3.3V: track 35.8 -> 69.5 mm, vias 0 -> 1
- net RESET: track 24.0 -> 0.00 mm
- net 5V: track 332.3 -> 312.8 mm
- net RAW: track 40.8 -> 56.3 mm
- net GND: track 18.0 -> 10.3 mm
- net N$17: track 10.4 -> 6.21 mm
- net N$18: track 7.28 -> 3.07 mm
- net N$1: track 1.88 -> 0.00 mm

Commit message: Further rearangement
Parts:
- moved J2 1.27 mm to (50.9, 30.5)
Routing:
- net 5V: track 312.8 -> 295.4 mm
- net 3.3V: track 69.5 -> 64.1 mm
- net GND: track 10.3 -> 5.67 mm
Changed lines of the file:
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@@
 <attribute name="PROD_ID" value="RES-07861" x="26.0985" y="32.512" size="1.778" layer="27" rot="R180" display="off"/>
 </element>
-<element name="J2" library="SparkFun-Connectors" package="2X3" value="AVR_SPI_PRG_6PTH" x="49.911" y="29.718" rot="MR0"/>
+<element name="J2" library="SparkFun-Connectors" package="2X3" value="AVR_SPI_PRG_6PTH" x="50.927" y="30.48" rot="MR0"/>
 <element name="U$1" library="LowPowerLab" package="RFM12B-ANTENNA" value="RFM12B_ANTENNA" x="45.5295" y="2.4765"/>
 <element name="U$5" library="LowPowerLab" package="RFM69W-MINPADS" value="RFM69" x="40.513" y="13.462" rot="MR270"/>
@@
 <contactref element="C31" pad="2"/>
 <contactref element="C32" pad="2"/>
-<wire x1="34.5095" y1="40.072" x2="33.528" y2="40.072" width="0.254" layer="1"/>
-<wire x1="33.528" y1="40.072" x2="33.528" y2="41.656" width="0.254" layer="1"/>
-<wire x1="33.528" y1="41.656" x2="35.381" y2="41.656" width="0.254" layer="1"/>
-<wire x1="35.381" y1="41.656" x2="35.381" y2="41.4365" width="0.254" layer="1"/>
 <wire x1="37.353" y1="34.2865" x2="37.353" y2="32.742" width="0.254" layer="1"/>
 <wire x1="37.353" y1="32.742" x2="36.107" y2="31.496" width="0.254" layer="1"/>
@@
 <wire x1="32.406" y1="36.128" x2="31.877" y2="35.599" width="0.254" layer="1"/>
 <wire x1="37.846" y1="38.1" x2="41.1825" y2="37.114" width="0" layer="19" extent="1-1"/>
+<wire x1="34.5095" y1="40.072" x2="35.381" y2="41.4365" width="0" layer="19" extent="1-1"/>
 <wire x1="5.7912" y1="35.403" x2="5.714" y2="30.644" width="0" layer="19" extent="1-1"/>
-<wire x1="53.848" y1="23.2782" x2="54.32308125" y2="15.518940625" width="0" layer="19" extent="1-1"/>
 </signal>
 <signal name="5V">
@@
 <wire x1="16.764" y1="50.8" x2="16.764" y2="48.006" width="1.27" layer="1"/>
 <wire x1="16.764" y1="48.006" x2="18.034" y2="46.736" width="1.27" layer="1"/>
-<wire x1="34.5095" y1="35.635" x2="35.306" y2="35.635" width="0.254" layer="1"/>
-<wire x1="35.306" y1="35.635" x2="35.306" y2="40.64" width="0.254" layer="1"/>
-<wire x1="35.306" y1="40.64" x2="34.5095" y2="40.64" width="0.254" layer="1"/>
-<wire x1="34.5095" y1="40.64" x2="34.5095" y2="40.565" width="0.254" layer="1"/>
-<wire x1="39.818" y1="41.4365" x2="39.818" y2="40.64" width="0.254" layer="1"/>
-<wire x1="39.818" y1="40.64" x2="35.306" y2="40.64" width="0.254" layer="1"/>
-<wire x1="41.1825" y1="36.621" x2="39.818" y2="36.621" width="0.254" layer="1"/>
-<wire x1="39.818" y1="36.621" x2="39.818" y2="40.64" width="0.254" layer="1"/>
 <wire x1="18.034" y1="46.736" x2="22.098" y2="42.672" width="1.27" layer="1"/>
 <wire x1="22.098" y1="42.672" x2="22.153" y2="42.617" width="1.27" layer="1"/>
@@
 <wire x1="26.67" y1="42.617" x2="26.67" y2="36.576" width="0.8128" layer="1"/>
 <wire x1="26.67" y1="36.576" x2="32.258" y2="30.988" width="0.8128" layer="1"/>
+<wire x1="50.927" y1="33.02" x2="48.7435" y2="35.814" width="0" layer="19" extent="1-1"/>
 <wire x1="41.6755" y1="36.621" x2="48.7435" y2="35.814" width="0" layer="19" extent="1-1"/>
+<wire x1="39.818" y1="41.4365" x2="41.1825" y2="36.621" width="0" layer="19" extent="1-1"/>
+<wire x1="34.5095" y1="40.565" x2="39.818" y2="41.4365" width="0" layer="19" extent="1-1"/>
+<wire x1="34.5095" y1="35.635" x2="34.5095" y2="40.565" width="0" layer="19" extent="1-1"/>
 <wire x1="32.258" y1="30.988" x2="34.0165" y2="35.635" width="0" layer="19" extent="1-1"/>
-<wire x1="49.911" y1="32.258" x2="48.7435" y2="35.814" width="0" layer="19" extent="1-1"/>
 </signal>
 <signal name="N$2">
@@
 <contactref element="S1" pad="3"/>
 <wire x1="50.4435" y1="35.814" x2="51.435" y2="38.1" width="0" layer="19" extent="1-1"/>
-<wire x1="41.6755" y1="36.128" x2="50.4435" y2="35.814" width="0" layer="19" extent="1-1"/>
-<wire x1="44.831" y1="29.718" x2="41.6755" y2="36.128" width="0" layer="19" extent="1-1"/>
+<wire x1="45.847" y1="30.48" x2="50.4435" y2="35.814" width="0" layer="19" extent="1-1"/>
+<wire x1="41.6755" y1="36.128" x2="45.847" y2="30.48" width="0" layer="19" extent="1-1"/>
 </signal>
 <signal name="SCK">
@@
 <contactref element="J2" pad="3"/>
 <contactref element="U$5" pad="SCK"/>
-<wire x1="47.371" y1="29.718" x2="39.325" y2="34.2865" width="0" layer="19" extent="1-1"/>
-<wire x1="41.513" y1="5.462" x2="47.371" y2="29.718" width="0" layer="19" extent="16-16"/>
+<wire x1="39.325" y1="34.2865" x2="48.387" y2="30.48" width="0" layer="19" extent="1-1"/>
+<wire x1="41.513" y1="5.462" x2="48.387" y2="30.48" width="0" layer="19" extent="16-16"/>
 </signal>
 <signal name="N$38">
@@
 <contactref element="J2" pad="1"/>
 <contactref element="U$5" pad="MISO"/>
-<wire x1="40.311" y1="34.2865" x2="49.911" y2="29.718" width="0" layer="19" extent="1-1"/>
-<wire x1="39.513" y1="5.462" x2="49.911" y2="29.718" width="0" layer="19" extent="16-16"/>
+<wire x1="40.311" y1="34.2865" x2="50.927" y2="30.48" width="0" layer="19" extent="1-1"/>
+<wire x1="39.513" y1="5.462" x2="50.927" y2="30.48" width="0" layer="19" extent="16-16"/>
 </signal>
 <signal name="MOSI">
@@
 <contactref element="J2" pad="4"/>
 <contactref element="U$5" pad="MOSI"/>
-<wire x1="47.371" y1="32.258" x2="39.818" y2="34.2865" width="0" layer="19" extent="1-1"/>
-<wire x1="37.513" y1="5.462" x2="47.371" y2="32.258" width="0" layer="19" extent="16-16"/>
+<wire x1="39.818" y1="34.2865" x2="48.387" y2="33.02" width="0" layer="19" extent="1-1"/>
+<wire x1="37.513" y1="5.462" x2="39.818" y2="34.2865" width="0" layer="19" extent="1-16"/>
 </signal>
 <signal name="RAW" class="1">
@@
 <wire x1="35.56" y1="46.228" x2="38.1" y2="48.768" width="1.27" layer="16"/>
 <wire x1="38.1" y1="48.768" x2="38.1" y2="50.8" width="1.27" layer="16"/>
-<wire x1="38.608" y1="53.594" x2="50.292" y2="53.594" width="0.8128" layer="1"/>
-<wire x1="50.292" y1="53.594" x2="52.832" y2="51.054" width="0.8128" layer="1"/>
-<wire x1="52.832" y1="51.054" x2="52.832" y2="24.638" width="0.8128" layer="1"/>
-<wire x1="38.608" y1="53.594" x2="38.1" y2="53.086" width="0.8128" layer="1"/>
-<wire x1="38.1" y1="53.086" x2="38.1" y2="50.8" width="0.8128" layer="1"/>
-<wire x1="52.832" y1="24.638" x2="49.442" y2="24.638" width="0.8128" layer="1"/>
 <wire x1="49.442" y1="24.638" x2="49.442" y2="22.479" width="0.8128" layer="1"/>
-<wire x1="52.832" y1="24.638" x2="52.832" y2="22.5942" width="0.254" layer="1"/>
-<wire x1="52.832" y1="22.5942" x2="53.848" y2="21.5782" width="0.254" layer="1"/>
 <wire x1="49.442" y1="24.638" x2="49.118" y2="24.962" width="0.8128" layer="1"/>
 <via x="49.118" y="24.962" extent="1-16" drill="0.6" shape="square"/>
 <wire x1="47.513" y1="24.962" x2="49.118" y2="24.962" width="0.8128" layer="16"/>
+<wire x1="38.1" y1="50.8" x2="38.1" y2="53.594" width="0.8128" layer="16"/>
+<wire x1="38.1" y1="53.594" x2="50.292" y2="53.594" width="0.8128" layer="16"/>
+<wire x1="50.292" y1="53.594" x2="52.832" y2="51.054" width="0.8128" layer="16"/>
+<wire x1="52.832" y1="51.054" x2="52.832" y2="28.702" width="0.8128" layer="16"/>
+<wire x1="52.832" y1="28.702" x2="49.118" y2="24.988" width="0.8128" layer="16"/>
+<wire x1="49.118" y1="24.988" x2="49.118" y2="24.962" width="0.8128" layer="16"/>
+<wire x1="49.442" y1="22.479" x2="53.848" y2="21.5782" width="0" layer="19" extent="1-1"/>
 </signal>
 <signal name="MPRIRQ">

Commit message: Initial autoroute
Routing:
- net 5V: track 295.4 -> 363.2 mm
- net SCK: track 0.00 -> 45.9 mm, vias 0 -> 2
- net USBVCC: track 5.00 -> 50.1 mm, vias 0 -> 2
- net MOSI: track 0.00 -> 40.5 mm, vias 0 -> 2
- net MISO: track 0.00 -> 40.0 mm, vias 0 -> 1
- net MPRIRQ: track 6.06 -> 41.4 mm, vias 0 -> 2
- net SDA: track 3.03 -> 37.7 mm, vias 0 -> 2
- net SS: track 0.00 -> 33.8 mm, vias 0 -> 1
- net D-: track 0.00 -> 31.6 mm, vias 0 -> 2
- net D+: track 0.00 -> 31.2 mm, vias 0 -> 2
- net SCL: track 4.38 -> 28.3 mm, vias 0 -> 4
- net RESET: track 0.00 -> 18.2 mm
- net RMFIRQ: track 0.00 -> 17.2 mm, vias 0 -> 1
- net GND: track 5.67 -> 19.9 mm
- net D10/LEDS: track 0.00 -> 14.0 mm, vias 0 -> 2
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
Commit message: Autorouted and DRC'd.  1st version sent to PCB
Parts:
- renumbered J2 to ISP, JP3 to CAPSENSORS, U$5 to RMF69
Other:
- board text added: "1kΩ"
- board text added: "220Ω"
- board text added: "22Ω"
