File: 32u4 plus 16LEDs/FabDisPendant.sch (EAGLE design)
At the start: 57 parts, among them U2 MIC5219, U3 ATMEGA32U4, Y1 16MHz

Commit message: Initial ATMega32u4 based pendant
Parts:
- removed D1: Yellow, SparkFun:LED0603
- added C26: 100uF, SparkFun-Capacitors:100UF-63V-20%(ELECT)
- added C27, C28: 0.1uF, SparkFun:CAP0603-CAP
- added FRAME3: FRAME-LEDGER, SparkFun-Aesthetics:FRAME-LEDGER
- added IC1: MPR121, Testing:MPR121V2
- added J2: AVR_SPI_PRG_6PTH, SparkFun-Connectors:AVR_SPI_PRG_6PTH
- added JP3: Electrodes, SparkFun:M12PTH
- added R1: 75k, SparkFun:RESISTOR0603-RES
- added R3, R9: 4.7k, SparkFun:RESISTOR0603-RES
- added R8: 220, SparkFun-Resistors:220OHM-1/10W-1%(0603)
- added U$1: RFM12B_ANTENNA, LowPowerLab:RFM12B_ANTENNA
- added U$5: RFM69, LowPowerLab:RFM69
- R4: value 330 -> 4.7k
Connections:
- removed net D10: L1.DIN, U3.PB6(ADC13)
- removed net D14: R4.1, U3.PB3(MISO)
- removed net D2: U3.PD1(SDA)
- removed net D3: U3.PD0(SCL)
- removed net N$23: D1.C, R4.2
- removed net RXI: U3.PD2(RX)
- removed net TXO: U3.PD3(TX)
- new net 3.3V: C28.1, IC1.VDD, R3.2, R4.2, R9.2
- new net ADDR: IC1.ADDR
- new net D10/LEDS: R8.1, U3.PB6(ADC13)
- new net ELE0: IC1.ELE0, JP3.12
- new net ELE1: IC1.ELE1, JP3.11
- new net ELE10: IC1.ELE10/LED6, JP3.2
- new net ELE11: IC1.ELE11/LED7, JP3.1
- new net ELE2: IC1.ELE2, JP3.10
- new net ELE3: IC1.ELE3, JP3.9
- new net ELE4: IC1.ELE4/LED0, JP3.8
- new net ELE5: IC1.ELE5/LED1, JP3.7
- new net ELE6: IC1.ELE6/LED2, JP3.6
- new net ELE7: IC1.ELE7/LED3, JP3.5
- new net ELE8: IC1.ELE8/LED4, JP3.4
- new net ELE9: IC1.ELE9/LED5, JP3.3
- new net MPRIRQ: IC1.~IRQ, R9.1, U3.PD3(TX)
- new net N$1: L1.DIN, R8.2
- new net N$25: U$1.1, U$5.ANT
- new net REXT: IC1.REXT, R1.2
- new net RMFIRQ: U$5.DIO0, U3.PD2(RX)
- new net SCL: IC1.SCL, R4.1, U3.PD0(SCL)
- new net SDA: IC1.SDA, R3.1, U3.PD1(SDA)
- new net SS: U$5.SEL, U3.PB3(MISO)
- new net VREG: C27.1, IC1.VREG
- net GND: now also C26.-, C27.2, C28.2, IC1.VSS, J2.6, R1.1, U$5.GND
- net MISO: now also J2.1, U$5.MISO
- net MOSI: now also J2.4, U$5.MOSI
- net RESET: now also J2.5
- net SCK: now also J2.3, U$5.SCK
- net VCC: now also C26.+, J2.2, U$5.VCC; no longer D1.A
Other:
- note added: "ISP Programming"
- note added: "LEDs"
- note added: "Power"
- note added: "Radio"
- note added: "USB"
- note removed: "Not used"
- moved on the sheet: C1, C10, C11, C12, C13, C14, C15, C16, C17, C18, C19, C2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

Commit message: Routed MPR121 and USB
Parts:
- removed FRAME3: FRAME-LEDGER, SparkFun-Aesthetics:FRAME-LEDGER
- removed SJ1: Closed for 5V Board, SparkFun:SOLDERJUMPERNC
- added S1: Reset, SparkFun:SWITCH-MOMENTARY-2SMD
Connections:
- net ELE0 renamed CAP0
- net ELE1 renamed CAP1
- net ELE10 renamed CAP10
- net ELE11 renamed CA011
- net ELE2 renamed CAP2
- net ELE3 renamed CAP3
- net ELE4 renamed CAP4
- net ELE5 renamed CAP5
- net ELE6 renamed CAP6
- net ELE7 renamed CAP7
- net ELE8 renamed CAP8
- net ELE9 renamed CAP9
- net UVCC renamed USBVCC
- removed net N$22: D2.A, F1.2, SJ1.1
- removed net VCC: C1.1, C10.1, C11.1, C12.1, C13.1, C14.1, C15.1, C16.1, C17.1, C18.+, C19.2, C2.1, C26.+, C3.1, C4.1, C5.1, C6.1, C7.1, C8.1, C9.1, D3.A, J2.2, L1.VDD, L10.VDD, L11.VDD, L12.VDD, L13.VDD, L14.VDD, L15.VDD, L16.VDD, L2.VDD, L3.VDD, L4.VDD, L5.VDD, L6.VDD, L7.VDD, L8.VDD, L9.VDD, R11.2, R2.2, SJ1.2, U$5.VCC, U2.OUT, U3.AVCC@24, U3.AVCC@44, U3.VCC@14, U3.VCC@34
- new net 5V: C1.1, C10.1, C11.1, C12.1, C13.1, C14.1, C15.1, C16.1, C17.1, C18.+, C19.2, C2.1, C26.+, C3.1, C4.1, C5.1, C6.1, C7.1, C8.1, C9.1, D2.A, D3.A, F1.2, J2.2, L1.VDD, L10.VDD, L11.VDD, L12.VDD, L13.VDD, L14.VDD, L15.VDD, L16.VDD, L2.VDD, L3.VDD, L4.VDD, L5.VDD, L6.VDD, L7.VDD, L8.VDD, L9.VDD, R11.2, R2.2, U2.OUT, U3.AVCC@24, U3.AVCC@44, U3.VCC@14, U3.VCC@34
- net 3.3V: now also U$5.VCC
- net GND: now also S1.1
- net RESET: now also S1.2
Other:
- note added: "Capacitive Touch"
- note added: "Need both 5 and 3.3V!"
- note added: "VCC = 5V"
- note removed: "Board is marked with combination of"
- note removed: "Open for 3.3V Board"
- note removed: "VCC = 5V or 3.3V Output"
- note removed: "resonator frequency and regulator voltage."
- moved on the sheet: C27, C28, IC1, JP3, R1, R2, R3, R4, R9

Commit message: Switch to 7805 regulator
Parts:
- removed C17: 1uF, SparkFun:CAP0603-CAP
- removed C18, C21: 10uF, SparkFun:CAP_POL1206
- removed C19: 0.1uF, SparkFun:CAP0603-CAP
- removed U2: MIC5219, SparkFun:V_REG_LDOSMD
- added 7803-???, 7805: 7805TV, linear:7805TV
- added C29, C31: 10uf, SparkFun-Capacitors:CAP_POLPTH2
- added C30, C32: 1uf, SparkFun-Capacitors:CAP_POLPTH2
- added PWR: M025MM, SparkFun-Connectors:M025MM
Connections:
- net 3.3V: now also 7803-???.GND, C32.+
- net 5V: now also 7805.VO, C30.+; no longer C17.1, C18.+, C19.2, U2.OUT
- net GND: now also 7803-???.VI, 7805.GND, C29.-, C30.-, C31.-, C32.-, PWR.2; no longer C17.2, C18.-, C19.1, C21.-, U2.GND
- net RAW: now also 7803-???.VO, 7805.VI, C29.+, C31.+, PWR.1; no longer C21.+, U2.EN, U2.IN
Other:
- note removed: "Need both 5 and 3.3V!"
- moved on the sheet: D2, F1, LED1, R11

Commit message: Checkin prior to autorouting
Parts:
- removed D3: Green, SparkFun:LED0603
- removed R6: 330, SparkFun:RESISTOR0603-RES
Connections:
- removed net N$24: D3.C, R6.2
- removed net TXLED: R6.1, U3.PD5
- net 5V: no longer D3.A
Changed lines of the file:
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@@
 <part name="C20" library="SparkFun" deviceset="CAP" device="0603-CAP" value="0.1uF"/>
 <part name="GND37" library="SparkFun" deviceset="GND" device=""/>
-<part name="R6" library="SparkFun" deviceset="RESISTOR" device="0603-RES" value="330"/>
-<part name="D3" library="SparkFun" deviceset="LED" device="0603" value="Green"/>
 <part name="P+11" library="SparkFun" deviceset="3.3V" device="" value="VCC"/>
 <part name="5V" library="SparkFun" deviceset="3.3V" device="" value="VCC"/>
@@
 <part name="F1" library="SparkFun" deviceset="PTC" device="SMD" value="500mA"/>
 <part name="D2" library="SparkFun" deviceset="DIODE" device="SOD"/>
-<part name="P+1" library="SparkFun" deviceset="VCC" device=""/>
 <part name="C26" library="SparkFun-Capacitors" deviceset="100UF-63V-20%(ELECT)" device="" value="100uF"/>
 <part name="R8" library="SparkFun-Resistors" deviceset="220OHM-1/10W-1%(0603)" device="" value="220"/>
@@
 </instance>
 <instance part="GND37" gate="1" x="162.56" y="119.38"/>
-<instance part="R6" gate="G$1" x="215.9" y="68.58" rot="R270"/>
-<instance part="D3" gate="G$1" x="215.9" y="55.88" smashed="yes" rot="R180">
-<attribute name="NAME" x="221.742" y="56.134" size="1.778" layer="95" rot="R90"/>
-<attribute name="VALUE" x="212.217" y="58.166" size="1.778" layer="96" rot="R270"/>
-</instance>
 <instance part="P+11" gate="G$1" x="167.64" y="165.1" smashed="yes">
 <attribute name="VALUE" x="165.354" y="168.402" size="1.778" layer="96"/>
@@
 <instance part="F1" gate="G$1" x="22.86" y="205.74"/>
 <instance part="D2" gate="G$1" x="40.64" y="205.74"/>
-<instance part="P+1" gate="1" x="215.9" y="50.8" rot="R180"/>
 <instance part="C26" gate="G$1" x="22.606" y="256.54" rot="R270"/>
 <instance part="R8" gate="G$1" x="16.891" y="245.618"/>
@@
 </segment>
 <segment>
-<wire x1="76.2" y1="198.12" x2="88.9" y2="198.12" width="0.1524" layer="91"/>
-<wire x1="88.9" y1="198.12" x2="88.9" y2="203.2" width="0.1524" layer="91"/>
-<wire x1="88.9" y1="198.12" x2="88.9" y2="195.58" width="0.1524" layer="91"/>
-<junction x="88.9" y="198.12"/>
-<pinref part="5V" gate="G$1" pin="3.3V"/>
-<pinref part="R11" gate="G$1" pin="2"/>
 <wire x1="30.48" y1="205.74" x2="33.02" y2="205.74" width="0.1524" layer="91"/>
 <wire x1="33.02" y1="205.74" x2="38.1" y2="205.74" width="0.1524" layer="91"/>
-<wire x1="33.02" y1="205.74" x2="33.02" y2="213.36" width="0.1524" layer="91"/>
+<wire x1="33.02" y1="205.74" x2="33.02" y2="215.9" width="0.1524" layer="91"/>
 <junction x="33.02" y="205.74"/>
 <pinref part="F1" gate="G$1" pin="2"/>
 <pinref part="D2" gate="G$1" pin="A"/>
-<wire x1="33.02" y1="213.36" x2="76.2" y2="213.36" width="0.1524" layer="91"/>
-<wire x1="76.2" y1="213.36" x2="76.2" y2="198.12" width="0.1524" layer="91"/>
-<wire x1="71.12" y1="198.12" x2="76.2" y2="198.12" width="0.1524" layer="91"/>
-<pinref part="C30" gate="G$1" pin="+"/>
-<wire x1="76.2" y1="193.04" x2="76.2" y2="198.12" width="0.1524" layer="91"/>
-<pinref part="7805" gate="A1" pin="VO"/>
-<junction x="76.2" y="198.12"/>
-<label x="72.136" y="198.374" size="1.778" layer="95"/>
-</segment>
-<segment>
-<wire x1="215.9" y1="50.8" x2="215.9" y2="53.34" width="0.1524" layer="91"/>
-<pinref part="D3" gate="G$1" pin="A"/>
-<pinref part="P+1" gate="1" pin="VCC"/>
+<wire x1="33.02" y1="215.9" x2="76.2" y2="215.9" width="0.1524" layer="91"/>
+<wire x1="76.2" y1="198.12" x2="76.2" y2="215.9" width="0.1524" layer="91"/>
 </segment>
 <segment>
@@
 <wire x1="83.82" y1="134.62" x2="91.44" y2="134.62" width="0.1524" layer="91"/>
 <wire x1="91.44" y1="134.62" x2="91.44" y2="142.24" width="0.1524" layer="91"/>
+</segment>
+<segment>
+<pinref part="R11" gate="G$1" pin="2"/>
+<pinref part="5V" gate="G$1" pin="3.3V"/>
+<wire x1="88.9" y1="198.12" x2="88.9" y2="203.2" width="0.1524" layer="91"/>
+<wire x1="88.9" y1="198.12" x2="88.9" y2="195.58" width="0.1524" layer="91"/>
+<junction x="88.9" y="198.12"/>
+<wire x1="76.2" y1="198.12" x2="88.9" y2="198.12" width="0.1524" layer="91"/>
+<pinref part="C30" gate="G$1" pin="+"/>
+<wire x1="76.2" y1="193.04" x2="76.2" y2="198.12" width="0.1524" layer="91"/>
+<junction x="76.2" y="198.12"/>
+<wire x1="71.12" y1="198.12" x2="76.2" y2="198.12" width="0.1524" layer="91"/>
+<pinref part="7805" gate="A1" pin="VO"/>
+<label x="72.136" y="198.374" size="1.778" layer="95"/>
 </segment>
 </net>
@@
 </segment>
 </net>
-<net name="TXLED" class="0">
-<segment>
-<wire x1="213.36" y1="76.2" x2="215.9" y2="76.2" width="0.1524" layer="91"/>
-<wire x1="215.9" y1="76.2" x2="215.9" y2="73.66" width="0.1524" layer="91"/>
-<pinref part="U3" gate="G$1" pin="PD5"/>
-<pinref part="R6" gate="G$1" pin="1"/>
-</segment>
-</net>
 <net name="N$20" class="0">
 <segment>
@@
 </segment>
 </net>
-<net name="N$24" class="0">
-<segment>
-<wire x1="215.9" y1="60.96" x2="215.9" y2="63.5" width="0.1524" layer="91"/>
-<pinref part="R6" gate="G$1" pin="2"/>
-<pinref part="D3" gate="G$1" pin="C"/>
-</segment>
-</net>

Commit message: Autorouted and DRC'd.  1st version sent to PCB
Parts:
- renumbered J2 to ISP, JP3 to CAPSENSORS, U$5 to RMF69
Changed lines of the file:
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@@
 <setting verticaltext="up"/>
 </settings>
-<grid distance="0.1" unitdist="inch" unit="inch" style="lines" multiple="1" display="no" altdistance="0.025" altunitdist="inch" altunit="inch"/>
+<grid distance="0.1" unitdist="inch" unit="inch" style="lines" multiple="1" display="no" altdistance="0.01" altunitdist="inch" altunit="inch"/>
 <layers>
 <layer number="1" name="Top" color="4" fill="1" visible="no" active="no"/>
@@
 <part name="R8" library="SparkFun-Resistors" deviceset="220OHM-1/10W-1%(0603)" device="" value="220"/>
 <part name="GND3" library="SparkFun-Aesthetics" deviceset="GND" device=""/>
-<part name="J2" library="SparkFun-Connectors" deviceset="AVR_SPI_PRG_6" device="PTH"/>
+<part name="ISP" library="SparkFun-Connectors" deviceset="AVR_SPI_PRG_6" device="PTH"/>
 <part name="SUPPLY2" library="SparkFun-Aesthetics" deviceset="VCC" device=""/>
 <part name="GND45" library="SparkFun-Aesthetics" deviceset="GND" device=""/>
@@
 <part name="P+3" library="SparkFun" deviceset="VCC" device="" value="3.3V"/>
 <part name="U$1" library="LowPowerLab" deviceset="RFM12B_ANTENNA" device=""/>
-<part name="U$5" library="LowPowerLab" deviceset="RFM69" device=""/>
+<part name="RMF69" library="LowPowerLab" deviceset="RFM69" device=""/>
 <part name="IC1" library="Testing" deviceset="MPR121" device="V2" value="MPR121"/>
 <part name="C27" library="SparkFun" deviceset="CAP" device="0603-CAP" value="0.1uF"/>
@@
 <part name="GND49" library="SparkFun" deviceset="GND" device=""/>
 <part name="C28" library="SparkFun" deviceset="CAP" device="0603-CAP" value="0.1uF"/>
-<part name="JP3" library="SparkFun" deviceset="M12" device="PTH" value="Electrodes"/>
+<part name="CAPSENSORS" library="SparkFun" deviceset="M12" device="PTH" value="Electrodes"/>
 <part name="R3" library="SparkFun" deviceset="RESISTOR" device="0603-RES" value="4.7k"/>
 <part name="R4" library="SparkFun" deviceset="RESISTOR" device="0603-RES" value="4.7k"/>
@@
 <instance part="R8" gate="G$1" x="16.891" y="245.618"/>
 <instance part="GND3" gate="1" x="13.208" y="256.54" rot="R270"/>
-<instance part="J2" gate="G$1" x="73.66" y="132.08"/>
+<instance part="ISP" gate="G$1" x="73.66" y="132.08"/>
 <instance part="SUPPLY2" gate="G$1" x="91.44" y="142.24"/>
 <instance part="GND45" gate="1" x="91.44" y="116.84"/>
@@
 <instance part="P+3" gate="1" x="334.01" y="144.78"/>
 <instance part="U$1" gate="G$1" x="346.71" y="146.05" rot="R90"/>
-<instance part="U$5" gate="G$1" x="334.01" y="125.73"/>
+<instance part="RMF69" gate="G$1" x="334.01" y="125.73"/>
 <instance part="IC1" gate="G$1" x="304.8" y="185.42"/>
 <instance part="C27" gate="G$1" x="266.7" y="172.72" smashed="yes">
@@
 <attribute name="NAME" x="255.524" y="203.581" size="1.778" layer="95"/>
 </instance>
-<instance part="JP3" gate="G$1" x="347.98" y="185.42" rot="R180"/>
+<instance part="CAPSENSORS" gate="G$1" x="347.98" y="185.42" rot="R180"/>
 <instance part="R3" gate="G$1" x="264.16" y="205.74" smashed="yes" rot="R90">
 <attribute name="NAME" x="266.2174" y="201.168" size="1.778" layer="95" rot="R90"/>
@@
 </segment>
 <segment>
-<pinref part="J2" gate="G$1" pin="6"/>
+<pinref part="ISP" gate="G$1" pin="6"/>
 <pinref part="GND45" gate="1" pin="GND"/>
 <wire x1="83.82" y1="129.54" x2="91.44" y2="129.54" width="0.1524" layer="91"/>
@@
 <wire x1="334.01" y1="113.03" x2="334.01" y2="115.57" width="0.1524" layer="91"/>
 <pinref part="SUPPLY18" gate="GND" pin="GND"/>
-<pinref part="U$5" gate="G$1" pin="GND"/>
+<pinref part="RMF69" gate="G$1" pin="GND"/>
 <junction x="334.01" y="113.03"/>
 </segment>
@@
 </segment>
 <segment>
-<pinref part="J2" gate="G$1" pin="2"/>
+<pinref part="ISP" gate="G$1" pin="2"/>
 <pinref part="SUPPLY2" gate="G$1" pin="VCC"/>
 <wire x1="83.82" y1="134.62" x2="91.44" y2="134.62" width="0.1524" layer="91"/>
@@
 </segment>
 <segment>
-<pinref part="J2" gate="G$1" pin="5"/>
+<pinref part="ISP" gate="G$1" pin="5"/>
 <wire x1="66.04" y1="129.54" x2="53.34" y2="129.54" width="0.1524" layer="91"/>
 <label x="53.34" y="129.54" size="1.778" layer="95"/>
@@
 </segment>
 <segment>
-<pinref part="J2" gate="G$1" pin="3"/>
+<pinref part="ISP" gate="G$1" pin="3"/>
 <wire x1="66.04" y1="132.08" x2="53.34" y2="132.08" width="0.1524" layer="91"/>
 <label x="53.34" y="132.08" size="1.778" layer="95"/>
@@
 <wire x1="306.07" y1="130.81" x2="321.31" y2="130.81" width="0.1524" layer="91"/>
 <label x="306.07" y="130.81" size="1.778" layer="95"/>
-<pinref part="U$5" gate="G$1" pin="SCK"/>
+<pinref part="RMF69" gate="G$1" pin="SCK"/>
 </segment>
 </net>
@@
 </segment>
 <segment>
-<pinref part="J2" gate="G$1" pin="1"/>
+<pinref part="ISP" gate="G$1" pin="1"/>
 <wire x1="66.04" y1="134.62" x2="53.34" y2="134.62" width="0.1524" layer="91"/>
 <label x="53.34" y="134.62" size="1.778" layer="95"/>
 </segment>
 <segment>
-<pinref part="U$5" gate="G$1" pin="MISO"/>
+<pinref part="RMF69" gate="G$1" pin="MISO"/>
 <wire x1="321.31" y1="128.27" x2="306.07" y2="128.27" width="0.1524" layer="91"/>
 <label x="306.07" y="128.27" size="1.778" layer="95"/>
@@
 </segment>
 <segment>
-<pinref part="J2" gate="G$1" pin="4"/>
+<pinref part="ISP" gate="G$1" pin="4"/>
 <wire x1="83.82" y1="132.08" x2="99.06" y2="132.08" width="0.1524" layer="91"/>
 <label x="93.98" y="132.08" size="1.778" layer="95"/>
 </segment>
 <segment>
-<pinref part="U$5" gate="G$1" pin="MOSI"/>
+<pinref part="RMF69" gate="G$1" pin="MOSI"/>
 <wire x1="321.31" y1="125.73" x2="306.07" y2="125.73" width="0.1524" layer="91"/>
 <label x="306.07" y="125.73" size="1.778" layer="95"/>
@@
 <wire x1="306.07" y1="133.35" x2="321.31" y2="133.35" width="0.1524" layer="91"/>
 <label x="306.07" y="133.35" size="1.778" layer="95"/>
-<pinref part="U$5" gate="G$1" pin="SEL"/>
+<pinref part="RMF69" gate="G$1" pin="SEL"/>
 </segment>
 <segment>
@@
 <pinref part="U$1" gate="G$1" pin="1"/>
 <wire x1="346.71" y1="140.97" x2="346.71" y2="128.27" width="0.1524" layer="91"/>
-<pinref part="U$5" gate="G$1" pin="ANT"/>
+<pinref part="RMF69" gate="G$1" pin="ANT"/>
 </segment>
 </net>
@@
 <label x="325.12" y="200.66" size="1.778" layer="95"/>
 <pinref part="IC1" gate="G$1" pin="ELE11/LED7"/>
-<pinref part="JP3" gate="G$1" pin="1"/>
+<pinref part="CAPSENSORS" gate="G$1" pin="1"/>
 </segment>
 </net>
@@
 <label x="325.12" y="198.12" size="1.778" layer="95"/>
 <pinref part="IC1" gate="G$1" pin="ELE10/LED6"/>
-<pinref part="JP3" gate="G$1" pin="2"/>
+<pinref part="CAPSENSORS" gate="G$1" pin="2"/>
 </segment>
 </net>
@@
 <label x="325.12" y="195.58" size="1.778" layer="95"/>
 <pinref part="IC1" gate="G$1" pin="ELE9/LED5"/>
-<pinref part="JP3" gate="G$1" pin="3"/>
+<pinref part="CAPSENSORS" gate="G$1" pin="3"/>
 </segment>
 </net>
@@
 <label x="325.12" y="193.04" size="1.778" layer="95"/>
 <pinref part="IC1" gate="G$1" pin="ELE8/LED4"/>
-<pinref part="JP3" gate="G$1" pin="4"/>
+<pinref part="CAPSENSORS" gate="G$1" pin="4"/>
 </segment>
 </net>
@@
 <label x="325.12" y="190.5" size="1.778" layer="95"/>
 <pinref part="IC1" gate="G$1" pin="ELE7/LED3"/>
-<pinref part="JP3" gate="G$1" pin="5"/>
+<pinref part="CAPSENSORS" gate="G$1" pin="5"/>
 </segment>
 </net>
@@
 <label x="325.12" y="187.96" size="1.778" layer="95"/>
 <pinref part="IC1" gate="G$1" pin="ELE6/LED2"/>
-<pinref part="JP3" gate="G$1" pin="6"/>
+<pinref part="CAPSENSORS" gate="G$1" pin="6"/>
 </segment>
 </net>
@@
 <label x="325.12" y="185.42" size="1.778" layer="95"/>
 <pinref part="IC1" gate="G$1" pin="ELE5/LED1"/>
-<pinref part="JP3" gate="G$1" pin="7"/>
+<pinref part="CAPSENSORS" gate="G$1" pin="7"/>
 </segment>
 </net>
@@
 <label x="325.12" y="182.88" size="1.778" layer="95"/>
 <pinref part="IC1" gate="G$1" pin="ELE4/LED0"/>
-<pinref part="JP3" gate="G$1" pin="8"/>
+<pinref part="CAPSENSORS" gate="G$1" pin="8"/>
 </segment>
 </net>
@@
 <label x="325.12" y="180.34" size="1.778" layer="95"/>
 <pinref part="IC1" gate="G$1" pin="ELE3"/>
-<pinref part="JP3" gate="G$1" pin="9"/>
+<pinref part="CAPSENSORS" gate="G$1" pin="9"/>
 </segment>
 </net>
@@
 <label x="325.12" y="177.8" size="1.778" layer="95"/>
 <pinref part="IC1" gate="G$1" pin="ELE2"/>
-<pinref part="JP3" gate="G$1" pin="10"/>
+<pinref part="CAPSENSORS" gate="G$1" pin="10"/>
 </segment>
 </net>
@@
 <label x="325.12" y="175.26" size="1.778" layer="95"/>
 <pinref part="IC1" gate="G$1" pin="ELE1"/>
-<pinref part="JP3" gate="G$1" pin="11"/>
+<pinref part="CAPSENSORS" gate="G$1" pin="11"/>
 </segment>
 </net>
@@
 <label x="325.12" y="172.72" size="1.778" layer="95"/>
 <pinref part="IC1" gate="G$1" pin="ELE0"/>
-<pinref part="JP3" gate="G$1" pin="12"/>
+<pinref part="CAPSENSORS" gate="G$1" pin="12"/>
 </segment>
 </net>
@@
 <pinref part="P+3" gate="1" pin="VCC"/>
 <wire x1="334.01" y1="144.78" x2="334.01" y2="140.97" width="0.1524" layer="91"/>
-<pinref part="U$5" gate="G$1" pin="VCC"/>
+<pinref part="RMF69" gate="G$1" pin="VCC"/>
 </segment>
 <segment>
@@
 <net name="RMFIRQ" class="0">
 <segment>
-<pinref part="U$5" gate="G$1" pin="DIO0"/>
+<pinref part="RMF69" gate="G$1" pin="DIO0"/>
 <wire x1="321.31" y1="120.65" x2="306.07" y2="120.65" width="0.1524" layer="91"/>
 <label x="306.07" y="120.65" size="1.778" layer="95"/>
