File: PCB/32u4 plus 16LEDs/FabDisPendant.brd (EAGLE design)
At the start: 76.2 x 54.2 mm, 68 parts, among them IC1 MPR121, U3 ATMEGA32U4, Y1 16MHz

Commit message: Continued improvement on the board design
Parts:
- moved C27 5.08 mm to (46.4, 15.4)
- moved IC1 5.08 mm to (50.0, 16.9)
- moved C28 5.08 mm to (48.8, 22.4)
- moved CAPSENSORS 5.08 mm to (55.5, 30.0)
- moved R1 5.08 mm to (48.9, 12.7)
- moved R3 5.08 mm to (45.2, 17.9)
- moved R4 5.08 mm to (45.2, 20.2)
- moved R9 5.08 mm to (45.2, 22.5)
Routing:
- net MPRIRQ: track 41.4 -> 29.1 mm
- net 3.3V: track 68.9 -> 72.9 mm
- net SDA: track 37.7 -> 41.7 mm
- net GND: track 19.9 -> 23.6 mm
- net SCL: track 28.3 -> 28.5 mm, vias 4 -> 2
Other:
- board size 76.2 x 54.2 mm -> 71.1 x 54.2 mm

Commit message: Switched from the TQDN package to an AU package
Parts:
- removed U3: ATMEGA32U4, Testing:QFN-44-NOPAD_1:1-OUTFAKES
- added U1: ATMEGA32U4-AU, Atmel_By_element14_Batch_1-00:QFP80P1200X1200X120-44N
Connections:
- removed net N$17: C23.1, U3.16, Y1.1
- removed net N$18: C22.1, U3.17, Y1.3
- removed net N$19: C24.2, U3.6
- new net D14: U1.22
- new net N$55: C24.2, U1.6
- new net XTAL1: C22.1, U1.17, Y1.3
- new net XTAL2: C23.1, U1.16, Y1.1
- net 5V: now also U1.14, U1.24, U1.34, U1.44; no longer U3.14, U3.24, U3.34, U3.44
- net A0: now also U1.36; no longer U3.36
- net A1: now also U1.37; no longer U3.37
- net A2: now also U1.38; no longer U3.38
- net A3: now also U1.39; no longer U3.39
- net A4: now also U1.40; no longer U3.40
- net A5: now also U1.41; no longer U3.41
- net AREF: now also U1.42; no longer U3.42
- net D+: now also U1.3; no longer U3.4
- net D-: now also U1.4; no longer U3.3
- net D10/LEDS: now also U1.30; no longer U3.30
- net D11: now also U1.12; no longer U3.12
- net D12: now also U1.26; no longer U3.26
- net D13: now also U1.32; no longer U3.32
- net D4: now also U1.25; no longer U3.25
- net D5: now also U1.31; no longer U3.31
- net D6: now also U1.27; no longer U3.27
- net D7: now also U1.1; no longer U3.1
- net D8: now also U1.28; no longer U3.28
- net D9: now also U1.29; no longer U3.29
- net GND: now also U1.15, U1.23, U1.33, U1.35, U1.43, U1.5; no longer U3.15, U3.23, U3.33, U3.35, U3.43, U3.5
- net MISO: now also U1.11; no longer U3.11
- net MOSI: now also U1.10; no longer U3.10
- net MPRIRQ: now also U1.21; no longer U3.21
- net RESET: now also U1.13; no longer U3.13
- net RMFIRQ: now also U1.20; no longer U3.20
- net SCK: now also U1.9; no longer U3.9
- net SCL: now also U1.18; no longer U3.18
- net SDA: now also U1.19; no longer U3.19
- net SS: now also U1.8; no longer U3.8
- net USBVCC: now also U1.2, U1.7; no longer U3.2, U3.7
Routing:
- net N$17: track 18.7 -> 0.00 mm
- net XTAL2: track 0.00 -> 18.2 mm
- net N$18: track 14.1 -> 0.00 mm
- net XTAL1: track 0.00 -> 12.2 mm
- net GND: track 23.6 -> 17.5 mm, vias 18 -> 17
- net 5V: track 362.8 -> 358.7 mm
- net N$19: track 2.81 -> 0.00 mm
- net SCL: track 28.5 -> 27.9 mm
- net SDA: track 41.7 -> 41.2 mm
- net RESET: track 18.2 -> 17.7 mm
