File: PCB/32u4_16LEDSMatrix/FabDisPendant.brd (EAGLE design)
At the start: 71.1 x 54.2 mm, 68 parts, among them IC1 MPR121, U1 ATMEGA32U4-AU, Y1 16MHz

Commit message: Completed switch to using 32u4 with the AU package
Parts:
- moved U1 56.6 mm to (39.6, 35.1), turned to 90 degrees
- moved R2 9.41 mm to (55.4, 43.2), turned to 270 degrees
- moved S1 8.86 mm to (53.6, 48.5)
- moved C24 5.85 mm to (39.6, 26.3), turned to 90 degrees
- moved U$1 5.68 mm to (50.6, 5.02)
- moved ISP 4.08 mm to (51.3, 34.5), turned to 90 degrees
- moved RMF69 3.31 mm to (40.8, 10.2)
- moved C20 2.30 mm to (32.1, 34.2), turned to 270 degrees
- moved Y1 1.57 mm to (47.2, 50.2)
- moved C22 1.57 mm to (45.7, 47.1)
- moved C23 1.57 mm to (49.0, 47.1)
Routing:
- net SDA: track 41.2 -> 26.0 mm
- net GND: track 17.5 -> 4.79 mm, vias 17 -> 19
- net 5V: track 358.7 -> 346.2 mm
- net 3.3V: track 72.9 -> 82.2 mm, vias 2 -> 1
- net D-: track 31.5 -> 38.3 mm
- net MOSI: track 40.5 -> 47.1 mm, vias 2 -> 1
- net XTAL1: track 12.2 -> 17.6 mm, vias 0 -> 2
- net N$25: track 2.99 -> 7.70 mm
- net USBVCC: track 50.1 -> 45.7 mm
- net SS: track 33.7 -> 29.4 mm
- net D+: track 31.2 -> 35.4 mm
- net SCL: track 27.9 -> 24.4 mm
- net RMFIRQ: track 17.2 -> 20.7 mm
- net XTAL2: track 18.2 -> 21.7 mm, vias 0 -> 2
- net D10/LEDS: track 13.9 -> 17.4 mm
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